File: hardware/carrier/carrier.kicad_sch (KiCad schematic)
At the start: 18 parts, among them J1 12V pigtail, U1 D1 Mini ESP32 (Type-C), U2 PCA9685 16ch servo, U3 LM2596 buck 12V->5.05V

Commit message: carrier V2: Scott's placement captured, outline restored, divider dropped, DRC 0
PCA on H3/H4 (its holes match the carrier's), D1 Mini in the left wing
with USB-C off the left edge, buck in the right wing, servo headers on
the bottom edge. No routing yet; V1's tracks belonged to the rejected
placement and are gone.

Why a capture step (gen/capture_placement.py -> placement.py) instead of
making the .kicad_pcb the master: the GUI-only path broke the outline
within one session (loose Edge.Cuts lines move under box-select) and
placed three parts off the real board. Regenerating keeps the DXF
outline, hole keepouts and D1 keepouts correct by construction.

Why the hole footprint lost its courtyard and silk ring, and the PCA
courtyard shrank to its header rows: the holes sit inside the PCA by
design; every DRC courtyard check was describing the intent.

Why solid pour connections on U2 pins 6/12 and U3 pins 2/4: servo and
buck return current, and the H3/H4 keepout leaves the PCA GND pins a
single 0.5 mm spoke. Everything else keeps thermal reliefs.

Why min_resolved_spokes 1: the D1's inner GND pin can only be reached
from the module middle; its other two GND pins carry the return.

Rail divider (R1/R2/TP4) removed per Scott: the ADC measured its own
noise, not sag.

Co-Authored-By: Claude Fable 5.1 <noreply@anthropic.com>
Parts:
- removed H4: M3 rack standoff, carrier:MountingHole_M3_3.175, symbol Mechanical:MountingHole
- removed R1: 10k, carrier:R_Axial_P10.16, symbol Device:R
- removed TP2: +5V, carrier:TestPoint_THT_D2.2_1.181, symbol Connector:TestPoint
- removed TP4: RAIL_ADC, carrier:TestPoint_THT_D2.2_1.181, symbol Connector:TestPoint
- added TP3: +3V3, carrier:TestPoint_THT_D2.2_1.181, symbol Connector:TestPoint
- H4: renamed from TP3; value +3V3 -> M3 rack standoff; footprint carrier:TestPoint_THT_D2.2_1.181 -> carrier:MountingHole_M3_3.175; symbol Connector:TestPoint -> Mechanical:MountingHole
- TP2: renamed from R2; value 10k -> +5V; footprint carrier:R_Axial_P10.16 -> carrier:TestPoint_THT_D2.2_1.181; symbol Device:R -> Connector:TestPoint
Connections:
- net +3V3: now also TP3.1; no longer H4.1
- net +5V: now also TP2.1
- net GND: no longer TP2.2
- net RAIL_ADC: no longer names the net of U1.4 (IO36)
- net RAIL_ADC: no longer TP2.1
- no-connect marks 30 -> 31
Other:
- note added: "Animatronic eyes carrier: D1 Mini ESP32 + PCA9685 + LM2596 on one milled board, M3 standoffs into the rack. Power: 12 V pigtail -> J1 -> LM2596 (set 5.0-5.1 V unloaded, USB unplugged) -> +5V. +5V is star-routed on the board: separate traces from U3 OUT+ to U2 V+ and to U1 VCC (pin 35). C1/C2 hang on the +5V run to U1 pin 35. No rail divider (dropped 2026-09-25: the on-board ADC only ever saw its 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"
- note removed: "Animatronic eyes carrier: D1 Mini ESP32 + PCA9685 + LM2596 on one milled board, M3 standoffs into the rack. Power: 12 V pigtail -> J1 -> LM2596 (set 5.0-5.1 V unloaded, USB unplugged) -> +5V. +5V is star-routed on the board: separate traces from U3 OUT+ to U2 V+ and to U1 VCC (pin 35). C1/C2 hang on the +5V run to U1 pin 35. R1/R2 divide the PCA V+ rail to GPIO36 (ADC1_CH0) for the rail monitor (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"

Commit message: carrier V2: routed single-sided, DRC 0/0/0, mill export + pcbmill drill check passed
All copper is in TRACKS in gen/gen_pcb.py (docstring there is the map). Pin decision:
SDA = IO27 (pad 24), SCL = IO25 (pad 26); firmware needs Wire.begin(27, 25) for the
carrier build (not changed here). IO21/22 are inner-row pins in Scott's placement and
the inner row's only exits are the module's USB end (already carrying +5V and +3V3)
and the antenna end - rejected.

Rejected alternatives, each of which DRC would have accepted:
- I2C to the PCA right row across the front bar: crosses the +3V3 lane.
- +3V3 down the far-left edge: fills the 1.35 mm strip that is GND's only path
  into the D1's middle (pad 33) and the back-left region (TP6).
- Feeding C1.1 by a stub from the y 10.9 run: walled off a GND pocket around C1.2
  that then hung on that pad's spoke alone (KiCad keeps pad-touching pour, so DRC
  says nothing) - now a diagonal off the lane, pour is one polygon + a 2 mm2 sliver.
- A +5V star to pad 35: would cross +3V3 or the GND entries into the left wing;
  V2 is a daisy chain OUT+ -> PCA V+ -> front bar -> left wing -> VCC.

Schematic: I2C nets moved to the PCA left row (3/4), right row keeps +5V/GND; the
jumper_pad_groups make either row valid. Stale V1 routing notes replaced.
export_for_mill.sh: DRC clean, gerbers, one merged drill (3 tools, 71 holes, all
exact bit sizes), annulus gate passed in a throwaway pcbmill job.

Co-Authored-By: Claude Fable 5.1 <noreply@anthropic.com>
Connections:
- net SCL: now also U1.26 (IO25), U2.4 (SCL); no longer U1.24 (IO27), U2.10 (SCL)
- net SDA: now also U1.24 (IO27), U2.3 (SDA); no longer U1.26 (IO25), U2.9 (SDA)
Other:
- note added: "Animatronic eyes carrier: D1 Mini ESP32 + PCA9685 + LM2596 on one milled board, M3 standoffs into the rack. Power: 12 V pigtail -> J1 -> LM2596 (set 5.0-5.1 V unloaded, USB unplugged) -> +5V. +5V: U3 OUT+ -> U2 V+ (right row) -> front-edge bar -> left wing -> C1/C2/U1 VCC (pin 35) via the USB end of U1. C1/C2 hang on the +5V run to U1 pin 35. No rail divider (dropped 2026-09-25: the on-board ADC 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"
- note removed: "Animatronic eyes carrier: D1 Mini ESP32 + PCA9685 + LM2596 on one milled board, M3 standoffs into the rack. Power: 12 V pigtail -> J1 -> LM2596 (set 5.0-5.1 V unloaded, USB unplugged) -> +5V. +5V is star-routed on the board: separate traces from U3 OUT+ to U2 V+ and to U1 VCC (pin 35). C1/C2 hang on the +5V run to U1 pin 35. No rail divider (dropped 2026-09-25: the on-board ADC only ever saw its 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"
Changed lines of the file:
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@@
 		)
 	)
-	(global_label "SCL"
+	(global_label "SDA"
 		(shape input)
 		(at 223.52 109.22 0)
@@
 		)
 	)
-	(global_label "SDA"
+	(global_label "SCL"
 		(shape input)
 		(at 223.52 114.3 0)
@@
 		)
 	)
-	(no_connect
-		(at 292.1 80.01)
-	)
-	(no_connect
-		(at 292.1 82.55)
+	(wire
+		(pts
+			(xy 292.1 80.01) (xy 287.02 80.01)
+		)
+		(stroke
+			(width 0)
+			(type default)
+		)
+	)
+	(global_label "SDA"
+		(shape input)
+		(at 287.02 80.01 180)
+		(fields_autoplaced yes)
+		(effects
+			(font
+				(size 1.27 1.27)
+			)
+			(justify right)
+		)
+		(property "Intersheetrefs" "${INTERSHEET_REFS}"
+			(at 287.02 80.01 0)
+			(hide yes)
+			(show_name no)
+			(do_not_autoplace no)
+			(effects
+				(font
+					(size 1.27 1.27)
+				)
+				(justify right)
+			)
+		)
+	)
+	(wire
+		(pts
+			(xy 292.1 82.55) (xy 287.02 82.55)
+		)
+		(stroke
+			(width 0)
+			(type default)
+		)
+	)
+	(global_label "SCL"
+		(shape input)
+		(at 287.02 82.55 180)
+		(fields_autoplaced yes)
+		(effects
+			(font
+				(size 1.27 1.27)
+			)
+			(justify right)
+		)
+		(property "Intersheetrefs" "${INTERSHEET_REFS}"
+			(at 287.02 82.55 0)
+			(hide yes)
+			(show_name no)
+			(do_not_autoplace no)
+			(effects
+				(font
+					(size 1.27 1.27)
+				)
+				(justify right)
+			)
+		)
 	)
 	(no_connect
@@
 		(at 317.5 77.47)
 	)
-	(wire
-		(pts
-			(xy 317.5 80.01) (xy 322.58 80.01)
-		)
-		(stroke
-			(width 0)
-			(type default)
-		)
-	)
-	(global_label "SDA"
-		(shape input)
-		(at 322.58 80.01 0)
-		(fields_autoplaced yes)
-		(effects
-			(font
-				(size 1.27 1.27)
-			)
-			(justify left)
-		)
-		(property "Intersheetrefs" "${INTERSHEET_REFS}"
-			(at 322.58 80.01 0)
-			(hide yes)
-			(show_name no)
-			(do_not_autoplace no)
-			(effects
-				(font
-					(size 1.27 1.27)
-				)
-				(justify left)
-			)
-		)
-	)
-	(wire
-		(pts
-			(xy 317.5 82.55) (xy 322.58 82.55)
-		)
-		(stroke
-			(width 0)
-			(type default)
-		)
-	)
-	(global_label "SCL"
-		(shape input)
-		(at 322.58 82.55 0)
-		(fields_autoplaced yes)
-		(effects
-			(font
-				(size 1.27 1.27)
-			)
-			(justify left)
-		)
-		(property "Intersheetrefs" "${INTERSHEET_REFS}"
-			(at 322.58 82.55 0)
-			(hide yes)
-			(show_name no)
-			(do_not_autoplace no)
-			(effects
-				(font
-					(size 1.27 1.27)
-				)
-				(justify left)
-			)
-		)
+	(no_connect
+		(at 317.5 80.01)
+	)
+	(no_connect
+		(at 317.5 82.55)
 	)
 	(no_connect
@@
 		)
 	)
-	(text "Animatronic eyes carrier: D1 Mini ESP32 + PCA9685 + LM2596 on one milled board, M3 standoffs into the rack.\nPower: 12 V pigtail -> J1 -> LM2596 (set 5.0-5.1 V unloaded, USB unplugged) -> +5V.\n+5V is star-routed on the board: separate traces from U3 OUT+ to U2 V+ and to U1 VCC (pin 35).\nC1/C2 hang on the +5V run to U1 pin 35. No rail divider (dropped 2026-09-25: the on-board ADC only ever saw its own noise).\nU2 rows are internally paralleled (jumper pad groups on the footprint), so either row can carry a net.\nI2C is on IO25 (SDA) / IO27 (SCL), not 21/22: single-sided routing can only reach the OUTER header columns. Wire.begin(25, 27).\nU1 pin numbers = header positions per r0oland ESP32_mini; VERIFY against the board silk before cutting."
+	(text "Animatronic eyes carrier: D1 Mini ESP32 + PCA9685 + LM2596 on one milled board, M3 standoffs into the rack.\nPower: 12 V pigtail -> J1 -> LM2596 (set 5.0-5.1 V unloaded, USB unplugged) -> +5V.\n+5V: U3 OUT+ -> U2 V+ (right row) -> front-edge bar -> left wing -> C1/C2/U1 VCC (pin 35) via the USB end of U1.\nC1/C2 hang on the +5V run to U1 pin 35. No rail divider (dropped 2026-09-25: the on-board ADC only ever saw its own noise).\nU2 rows are internally paralleled (jumper pad groups on the footprint), so either row can carry a net.\nI2C is on IO27 (SDA) / IO25 (SCL), not 21/22: single-sided routing can only reach the OUTER header columns. Wire.begin(27, 25).\nU1 pin numbers = header positions per r0oland ESP32_mini; VERIFY against the board silk before cutting."
 		(exclude_from_sim no)
 		(at 38.1 215.9 0)

Commit message: carrier: J1 at Scott's spot, C1 turned, schematic parity clean, STEP re-exported
Scott placed J1 at (45.05,15.7) between H4 and the chamfer after my move
left its body against the buck's IN- corner, and turned C1 so the TP2 stub
runs straight into it; that removes the diagonal and the pour sliver
(pour is one polygon). +12V goes east under J1 then north: straight north
from the new pad would graze IN- by 0.05.
The parity errors he saw were generator defects: NC pads without the
netlist's unconnected-() nets, symbol Description empty, Datasheet ~ vs
empty, and two different J1 values. Fixed at the source (gen_pcb/gen_sch)
rather than by excluding them in the .kicad_pro, so the check stays live.
docs STEP re-exported by kicad-cli after the rebuild - a GUI export from
before the rebuild was already stale.
ERC 0, DRC --schematic-parity 0/0/0, gerbers + drill re-exported, pcbmill
bit map exact + annulus gate passed.

Co-Authored-By: Claude Fable 5.1 <noreply@anthropic.com>
Parts:
- J1: value 12V pigtail -> 12V in
Changed lines of the file:
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@@
 			)
 		)
-		(property "Datasheet" "~"
+		(property "Datasheet" ""
 			(at 203.2 121.92 0)
 			(hide yes)
@@
 			)
 		)
-		(property "Description" ""
+		(property "Description" "D1 Mini ESP32 (WROOM-32), 40-pin, 1.78/1.181 pads, flash pins NPTH"
 			(at 203.2 121.92 0)
 			(hide yes)
@@
 			)
 		)
-		(property "Datasheet" "~"
+		(property "Datasheet" ""
 			(at 304.8 81.28 0)
 			(hide yes)
@@
 			)
 		)
-		(property "Description" ""
+		(property "Description" "PCA9685 16ch servo board (Adafruit rev C geometry), 2x 1x06 rows 58.42 mm apart, body 62.23 x 25.4"
 			(at 304.8 81.28 0)
 			(hide yes)
@@
 			)
 		)
-		(property "Datasheet" "~"
+		(property "Datasheet" ""
 			(at 101.6 81.28 0)
 			(hide yes)
@@
 			)
 		)
-		(property "Description" ""
+		(property "Description" "LM2596 buck module, 4 pins 17.6 x 39.8 mm (ratgdo footprint, NOT caliper-verified)"
 			(at 101.6 81.28 0)
 			(hide yes)
@@
 			)
 		)
-		(property "Value" "12V pigtail"
+		(property "Value" "12V in"
 			(at 50.8 86.36 0)
 			(show_name no)
@@
 			)
 		)
-		(property "Datasheet" "~"
+		(property "Datasheet" ""
 			(at 50.8 81.28 0)
 			(hide yes)
@@
 			)
 		)
-		(property "Description" ""
+		(property "Description" "KF301-5.0 screw terminal 2P 5.08 mm, pads 2.6/1.181"
 			(at 50.8 81.28 0)
 			(hide yes)
@@
 			)
 		)
-		(property "Datasheet" "~"
+		(property "Datasheet" ""
 			(at 101.6 139.7 0)
 			(hide yes)
@@
 			)
 		)
-		(property "Description" ""
+		(property "Description" "220 uF radial electrolytic, 6.3 dia, 2.5 pitch, pin 1 = +"
 			(at 101.6 139.7 0)
 			(hide yes)
@@
 			)
 		)
-		(property "Datasheet" "~"
+		(property "Datasheet" ""
 			(at 121.92 139.7 0)
 			(hide yes)
@@
 			)
 		)
-		(property "Description" ""
+		(property "Description" "100 nF ceramic disc/MLCC, 5.08 mm pitch (0.1 in leads)"
 			(at 121.92 139.7 0)
 			(hide yes)
@@
 			)
 		)
-		(property "Datasheet" "~"
+		(property "Datasheet" ""
 			(at 50.8 190.5 0)
 			(hide yes)
@@
 			)
 		)
-		(property "Description" ""
+		(property "Description" "Drilled test point, 2.2 pad on the 1.181 bit (0.51 annulus)"
 			(at 50.8 190.5 0)
 			(hide yes)
@@
 			)
 		)
-		(property "Datasheet" "~"
+		(property "Datasheet" ""
 			(at 63.5 190.5 0)
 			(hide yes)
@@
 			)
 		)
-		(property "Description" ""
+		(property "Description" "Drilled test point, 2.2 pad on the 1.181 bit (0.51 annulus)"
 			(at 63.5 190.5 0)
 			(hide yes)
@@
 			)
 		)
-		(property "Datasheet" "~"
+		(property "Datasheet" ""
 			(at 76.2 190.5 0)
 			(hide yes)
@@
 			)
 		)
-		(property "Description" ""
+		(property "Description" "Drilled test point, 2.2 pad on the 1.181 bit (0.51 annulus)"
 			(at 76.2 190.5 0)
 			(hide yes)
@@
 			)
 		)
-		(property "Datasheet" "~"
+		(property "Datasheet" ""
 			(at 101.6 190.5 0)
 			(hide yes)
@@
 			)
 		)
-		(property "Description" ""
+		(property "Description" "Drilled test point, 2.2 pad on the 1.181 bit (0.51 annulus)"
 			(at 101.6 190.5 0)
 			(hide yes)
@@
 			)
 		)
-		(property "Datasheet" "~"
+		(property "Datasheet" ""
 			(at 114.3 190.5 0)
 			(hide yes)
@@
 			)
 		)
-		(property "Description" ""
+		(property "Description" "Drilled test point, 2.2 pad on the 1.181 bit (0.51 annulus)"
 			(at 114.3 190.5 0)
 			(hide yes)
@@
 			)
 		)
-		(property "Datasheet" "~"
+		(property "Datasheet" ""
 			(at 269.24 190.5 0)
 			(hide yes)
@@
 			)
 		)
-		(property "Description" ""
+		(property "Description" "M3 rack standoff hole, drilled 3.175 (the bit), NPTH; pour keepout is a board rule area"
 			(at 269.24 190.5 0)
 			(hide yes)
@@
 			)
 		)
-		(property "Datasheet" "~"
+		(property "Datasheet" ""
 			(at 284.48 190.5 0)
 			(hide yes)
@@
 			)
 		)
-		(property "Description" ""
+		(property "Description" "M3 rack standoff hole, drilled 3.175 (the bit), NPTH; pour keepout is a board rule area"
 			(at 284.48 190.5 0)
 			(hide yes)
@@
 			)
 		)
-		(property "Datasheet" "~"
+		(property "Datasheet" ""
 			(at 299.72 190.5 0)
 			(hide yes)
@@
 			)
 		)
-		(property "Description" ""
+		(property "Description" "M3 rack standoff hole, drilled 3.175 (the bit), NPTH; pour keepout is a board rule area"
 			(at 299.72 190.5 0)
 			(hide yes)
@@
 			)
 		)
-		(property "Datasheet" "~"
+		(property "Datasheet" ""
 			(at 314.96 190.5 0)
 			(hide yes)
@@
 			)
 		)
-		(property "Description" ""
+		(property "Description" "M3 rack standoff hole, drilled 3.175 (the bit), NPTH; pour keepout is a board rule area"
 			(at 314.96 190.5 0)
 			(hide yes)
